File: memory-zif.sch (KiCad schematic (older format))
At the start: 10 parts, among them J1 Conn_01x30_Male, SW1 SW_DPDT_x2, U1 28C256, U2 74LS04, U3 HM62256BLP

Commit message: using 128K RAM rather than 32K RAM
Parts:
- removed J1: Conn_01x30_Male, Connector_PinHeader_2.54mm:PinHeader_1x30_P2.54mm_Vertical, symbol Connector:Conn_01x30_Male
- removed SW1: SW_DPDT_x2, Button_Switch_THT:SW_E-Switch_EG1271_DPDT, symbol Switch:SW_DPDT_x2
- removed U3: HM62256BLP, Package_DIP:DIP-28_W15.24mm_Socket_LongPads, symbol Memory_RAM:HM62256BLP
- added J1: ADDRESS, Connector_PinHeader_2.54mm:PinHeader_1x17_P2.54mm_Vertical, symbol Connector:Conn_01x17_Male
- added J2: DATA, Connector_PinHeader_2.54mm:PinHeader_1x08_P2.54mm_Vertical, symbol Connector:Conn_01x08_Male
- added J3: CONTROL, Connector_PinHeader_2.54mm:PinHeader_1x04_P2.54mm_Vertical, symbol Connector:Conn_01x04_Male
- added J4: POWER, Connector_PinHeader_2.54mm:PinHeader_1x02_P2.54mm_Vertical, symbol Connector:Conn_01x02_Male
- added R1, R3: 10K, Resistor_THT:R_Axial_DIN0204_L3.6mm_D1.6mm_P5.08mm_Horizontal, symbol Device:R_Small
- added SW1: SW_SPDT, Switches:SWITCH_SPDT_PTH_11.6X4.0MM, symbol Switch:SW_SPDT
- added U3: 628128, Package_DIP:DIP-32_W15.24mm_Socket_LongPads, symbol Memory_RAM:628128_DIP32_SSOP32
- U1: footprint Package_DIP:DIP-28_W15.24mm_Socket_LongPads -> Socket:DIP_Socket-28_W11.9_W12.7_W15.24_W17.78_W18.5_3M_228-1277-00-0602J
Connections:
- net ~WE is gone; now on net +5V: U1.27 (~WE)
- net +5V: now also J4.1 (Pin_1), R1.1, R3.1, U3.30 (CS2), U3.32 (VCC)
- net A0: now also J1.1 (Pin_1), U3.12 (A0)
- net A1: now also J1.2 (Pin_2), U3.11 (A1)
- net A10: now also J1.11 (Pin_11), U3.23 (A10)
- net A11: now also J1.12 (Pin_12), U3.25 (A11)
- net A12: now also J1.13 (Pin_13), U3.4 (A12)
- net A13: now also J1.14 (Pin_14), U3.28 (A13)
- net A14: now also J1.15 (Pin_15), U3.3 (A14)
- net A2: now also J1.3 (Pin_3), U3.10 (A2)
- net A3: now also J1.4 (Pin_4), U3.9 (A3)
- net A4: now also J1.5 (Pin_5), U3.8 (A4)
- net A5: now also J1.6 (Pin_6), U3.7 (A5)
- net A6: now also J1.7 (Pin_7), U3.6 (A6)
- net A7: now also J1.8 (Pin_8), U3.5 (A7)
- net A8: now also J1.9 (Pin_9), U3.27 (A8)
- net A9: now also J1.10 (Pin_10), U3.26 (A9)
- net D0: now also J2.1 (Pin_1), U3.13 (Q0)
- net D1: now also J2.2 (Pin_2), U3.14 (Q1)
- net D2: now also J2.3 (Pin_3), U3.15 (Q2)
- net D3: now also J2.4 (Pin_4), U3.17 (Q3)
- net D4: now also J2.5 (Pin_5), U3.18 (Q4)
- net D5: now also J2.6 (Pin_6), U3.19 (Q5)
- net D6: now also J2.7 (Pin_7), U3.20 (Q6)
- net D7: now also J2.8 (Pin_8), U3.21 (Q7)
- net GND: now also U1.22 (~OE), J4.2 (Pin_2), U3.16 (GND)
- net R~W: now also J3.4 (Pin_4), R3.2, U3.29 (~WE)
- net ~OE: now also SW1.2 (B), U3.24 (~OE); no longer U1.22 (~OE)
- net ~RAM: now also J3.2 (Pin_2), U3.22 (~CS1)
- net ~RD: now also J3.3 (Pin_3), R1.2, SW1.1 (A)
- net ~ROM: now also J3.1 (Pin_1)
- net ~R~W: now also SW1.3 (C)
- new net A15: J1.16 (Pin_16), U3.31 (A15)
- new net A16: J1.17 (Pin_17), U3.2 (A16)
